Commit message: Added lidar

File: src/smf1_description/urdf/mybot.xacro (robot description, xacro)
@@ -93,3 +93,31 @@
     </inertial>
   </link>
+  <xacro:include filename="$(find velodyne_description)/urdf/VLP-16.urdf.xacro"/>
+  <VLP-16 parent="mount" name="velodyne" topic="/velodyne_points" hz="10" samples="440">
+    <origin xyz="0 0 0.025" rpy="0 0 0" />
+  </VLP-16>
+  <joint name="mount" type="fixed" >
+   <parent link="chassis" />
+    <child link="mount" />
+    <origin xyz="0 0 ${0.05+wheelRadius+0.05/2}" rpy="0 0 0" />
+  </joint>
+  <link name="mount" >
+    <visual>
+      <geometry>
+        <box size="0.05 0.05 0.05" />
+      </geometry>
+    </visual>
+    <collision>
+      <geometry>
+        <box size="0.05 0.05 0.05" />
+      </geometry>
+    </collision>
+    <inertial>
+      <origin xyz="0 0 0"/>
+      <mass value="10"/>
+      <inertia ixx="3.0" ixy="0.0" ixz="0.0"
+               iyy="3.0" iyz="0.0"
+               izz="3.0" />
+    </inertial>
+  </link>
 </robot>

Commit message: smf1 lidar; Adjusted lidar distance and mount height.

File: src/smf1_description/urdf/mybot.xacro (robot description, xacro)
@@ -14,4 +14,5 @@
   <xacro:property name="cameraSize" value="0.05"/>
   <xacro:property name="cameraMass" value="0.1"/>
+  <xacro:property name="mount_height" value="0.08"/>
   <xacro:include filename="$(find smf1_description)/urdf/mybot.gazebo" />
   <xacro:include filename="$(find smf1_description)/urdf/materials.xacro" />
@@ -100,10 +101,10 @@
    <parent link="chassis" />
     <child link="mount" />
-    <origin xyz="0 0 ${0.05+wheelRadius+0.05/2}" rpy="0 0 0" />
+    <origin xyz="0 0 ${0.05+wheelRadius+mount_height/2}" rpy="0 0 0" />
   </joint>
   <link name="mount" >
     <visual>
       <geometry>
-        <box size="0.05 0.05 0.05" />
+        <box size="0.05 0.05 ${mount_height}" />
       </geometry>
     </visual>

File: src/velodyne_description/urdf/VLP-16.urdf.xacro (robot description, xacro)
@@ -2,5 +2,6 @@
 <robot xmlns:xacro="http://www.ros.org/wiki/xacro" name="VLP-16">
   <xacro:property name="M_PI" value="3.1415926535897931" />
-  <xacro:macro name="VLP-16" params="*origin parent:=base_link name:=velodyne topic:=/velodyne_points hz:=10 lasers:=16 samples:=1875 collision_range:=0.3 min_range:=0.9 max_range:=130.0 noise:=0.008 min_angle:=-${M_PI} max_angle:=${M_PI}">
+  <xacro:macro name="VLP-16" params="*origin parent:=base_link name:=velodyne topic:=/velodyne_points hz:=10 lasers:=16 samples:=1875
+  collision_range:=0.1 min_range:=0.1 max_range:=130.0 noise:=0.008 min_angle:=-${M_PI} max_angle:=${M_PI}">
     <joint name="${name}_base_mount_joint" type="fixed">
       <xacro:insert_block name="origin" />
